File: WatchDog/WatchDog.brd (EAGLE design)
At the start: 30.5 x 27.6 mm, 18 parts

Commit message: update
Routing:
- net N$14: vias 4 -> 6
- added copper zone on layer 1, net N$14
- added copper zone on layer 16, net N$14
- removed copper zone on layer 16, net GND
Changed lines of the file:
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@@
 <wire x1="30.366" y1="69.215" x2="31.001" y2="68.58" width="0.1524" layer="1"/>
 <wire x1="31.001" y1="68.58" x2="31.75" y2="68.58" width="0.1524" layer="1"/>
-<wire x1="34.29" y1="72.39" x2="34.29" y2="71.12" width="0.1524" layer="16"/>
-<wire x1="34.29" y1="71.12" x2="31.75" y2="68.58" width="0.1524" layer="16"/>
+<wire x1="34.29" y1="72.39" x2="34.29" y2="71.12" width="0.4064" layer="16"/>
+<wire x1="34.29" y1="71.12" x2="31.75" y2="68.58" width="0.4064" layer="16"/>
 <via x="34.29" y="78.74" extent="1-16" drill="0.35"/>
 <wire x1="34.29" y1="78.74" x2="33.782" y2="78.232" width="0.1524" layer="1"/>
 <wire x1="33.782" y1="78.232" x2="33.02" y2="78.232" width="0.1524" layer="1"/>
-<wire x1="34.29" y1="72.39" x2="34.29" y2="78.74" width="0.1524" layer="16"/>
-<wire x1="40.64" y1="78.232" x2="43.18" y2="78.232" width="0.1524" layer="1"/>
-<wire x1="43.18" y1="78.232" x2="44.45" y2="78.232" width="0.1524" layer="1"/>
-<wire x1="44.45" y1="78.232" x2="45.72" y2="78.232" width="0.1524" layer="1"/>
-<wire x1="45.72" y1="78.232" x2="47.498" y2="78.232" width="0.1524" layer="1"/>
-<wire x1="47.498" y1="78.232" x2="48.26" y2="77.47" width="0.1524" layer="1"/>
-<wire x1="48.26" y1="77.47" x2="46.99" y2="78.74" width="0.1524" layer="16"/>
-<wire x1="46.99" y1="78.74" x2="34.29" y2="78.74" width="0.1524" layer="16"/>
+<wire x1="34.29" y1="72.39" x2="34.29" y2="78.74" width="0.4064" layer="16"/>
+<wire x1="40.64" y1="78.232" x2="43.18" y2="78.232" width="0.508" layer="1"/>
+<wire x1="43.18" y1="78.232" x2="44.45" y2="78.232" width="0.508" layer="1"/>
+<wire x1="44.45" y1="78.232" x2="45.72" y2="78.232" width="0.508" layer="1"/>
+<wire x1="45.72" y1="78.232" x2="47.498" y2="78.232" width="0.508" layer="1"/>
+<wire x1="47.498" y1="78.232" x2="48.26" y2="77.47" width="0.508" layer="1"/>
+<wire x1="48.26" y1="77.47" x2="46.99" y2="78.74" width="0.4064" layer="16"/>
+<wire x1="46.99" y1="78.74" x2="34.29" y2="78.74" width="0.4064" layer="16"/>
 <wire x1="35.674" y1="73.015" x2="36.5727125" y2="73.015" width="0.1524" layer="1"/>
 <wire x1="39.2636" y1="72.4964" x2="39.37" y2="72.39" width="0.1524" layer="1"/>
@@
 <contactref element="C3" pad="1"/>
 <contactref element="NE555" pad="5"/>
-<wire x1="36.83" y1="78.232" x2="31.623" y2="73.025" width="0.1524" layer="1"/>
-<wire x1="31.623" y1="73.025" x2="30.366" y2="73.025" width="0.1524" layer="1"/>
+<wire x1="36.83" y1="78.232" x2="31.623" y2="73.025" width="0.4064" layer="1"/>
+<wire x1="31.623" y1="73.025" x2="30.366" y2="73.025" width="0.4064" layer="1"/>
 </signal>
 <signal name="N$1">
@@
 <wire x1="33.02" y1="63.5" x2="33.02" y2="64.77" width="1.016" layer="16"/>
 <wire x1="33.02" y1="63.5" x2="33.02" y2="59.69" width="1.016" layer="16"/>
+<polygon width="0.1524" layer="16">
+<vertex x="27.94" y="80.01"/>
+<vertex x="27.94" y="54.61"/>
+<vertex x="55.88" y="54.61"/>
+<vertex x="55.88" y="80.01"/>
+</polygon>
+<polygon width="0.1524" layer="1">
+<vertex x="55.88" y="54.61"/>
+<vertex x="55.88" y="80.01"/>
+<vertex x="27.94" y="80.01"/>
+<vertex x="27.94" y="54.61"/>
+</polygon>
+<via x="39.37" y="67.31" extent="1-16" drill="0.35"/>
+<via x="49.53" y="55.88" extent="1-16" drill="0.35"/>
 </signal>
 <signal name="N$2">
@@
 <wire x1="41.402" y1="57.15" x2="43.942" y2="57.15" width="0.1524" layer="1"/>
 </signal>
-<signal name="GND">
-<polygon width="0.1524" layer="16">
-<vertex x="27.94" y="80.01"/>
-<vertex x="27.94" y="54.61"/>
-<vertex x="55.88" y="54.61"/>
-<vertex x="55.88" y="80.01"/>
-</polygon>
+<signal name="N$5">
+<via x="31.75" y="78.74" extent="1-16" drill="0.35"/>
 </signal>
 </signals>

Commit message: update
Routing:
- net N$6: track 24.8 -> 42.3 mm, vias 3 -> 0
- net N$14: track 87.6 -> 70.6 mm, vias 6 -> 2
- net N$1: track 32.4 -> 38.1 mm
- net N$3: track 18.5 -> 15.2 mm, vias 3 -> 0
- net N$7: track 14.9 -> 14.2 mm
- net N$9: track 46.3 -> 46.9 mm
